Commit message: updated project code

File: assets/franka_description/robots/nugget.urdf (robot description, URDF)
Before this commit: robot nugget, 1 links, 0 joints
Links:
- link base_link: mass .017 -> .02; geometry collision mesh filename=package://scene/nugget_1.stl scale=0.001 0.001 0.001; visual mesh filename=package://scene/nugget_1.stl scale=0.001 0.001 0.001
